Commit message: docs: add dexterous hand mimic joints and execution troubleshooting

File: research/simulation/assets/robots/ar5_l6/urdf/left/ahmed_moveit/config/ar5_o6_left.ros2_control.xacro (robot description, xacro)
@@ -1,103 +1,102 @@
-<?xml version="1.0"?>
+<?xml version='1.0' encoding='us-ascii'?>
 <robot xmlns:xacro="http://www.ros.org/wiki/xacro">
     <xacro:macro name="ar5_o6_left_ros2_control" params="name initial_positions_file">
-        <xacro:property name="initial_positions" value="${xacro.load_yaml(initial_positions_file)['initial_positions']}"/>
+        <xacro:property name="initial_positions" value="${xacro.load_yaml(initial_positions_file)['initial_positions']}" />
         <ros2_control name="${name}" type="system">
             <hardware>
-                <!-- By default, set up controllers for simulation. This won't work on real hardware -->
                 <plugin>mock_components/GenericSystem</plugin>
             </hardware>
             <joint name="AR5_5_07L_W4C4A2_joint_1">
-                <command_interface name="position"/>
+                <command_interface name="position" />
                 <state_interface name="position">
                   <param name="initial_value">${initial_positions['AR5_5_07L_W4C4A2_joint_1']}</param>
                 </state_interface>
-                <state_interface name="velocity"/>
+                <state_interface name="velocity" />
             </joint>
             <joint name="AR5_5_07L_W4C4A2_joint_2">
-                <command_interface name="position"/>
+                <command_interface name="position" />
                 <state_interface name="position">
                   <param name="initial_value">${initial_positions['AR5_5_07L_W4C4A2_joint_2']}</param>
                 </state_interface>
-                <state_interface name="velocity"/>
+                <state_interface name="velocity" />
             </joint>
             <joint name="AR5_5_07L_W4C4A2_joint_3">
-                <command_interface name="position"/>
+                <command_interface name="position" />
                 <state_interface name="position">
                   <param name="initial_value">${initial_positions['AR5_5_07L_W4C4A2_joint_3']}</param>
                 </state_interface>
-                <state_interface name="velocity"/>
+                <state_interface name="velocity" />
             </joint>
             <joint name="AR5_5_07L_W4C4A2_joint_4">
-                <command_interface name="position"/>
+                <command_interface name="position" />
                 <state_interface name="position">
                   <param name="initial_value">${initial_positions['AR5_5_07L_W4C4A2_joint_4']}</param>
                 </state_interface>
-                <state_interface name="velocity"/>
+                <state_interface name="velocity" />
             </joint>
             <joint name="AR5_5_07L_W4C4A2_joint_5">
-                <command_interface name="position"/>
+                <command_interface name="position" />
                 <state_interface name="position">
                   <param name="initial_value">${initial_positions['AR5_5_07L_W4C4A2_joint_5']}</param>
                 </state_interface>
-                <state_interface name="velocity"/>
+                <state_interface name="velocity" />
             </joint>
             <joint name="AR5_5_07L_W4C4A2_joint_6">
-                <command_interface name="position"/>
+                <command_interface name="position" />
                 <state_interface name="position">
                   <param name="initial_value">${initial_positions['AR5_5_07L_W4C4A2_joint_6']}</param>
                 </state_interface>
-                <state_interface name="velocity"/>
+                <state_interface name="velocity" />
             </joint>
             <joint name="AR5_5_07L_W4C4A2_joint_7">
-                <command_interface name="position"/>
+                <command_interface name="position" />
                 <state_interface name="position">
                   <param name="initial_value">${initial_positions['AR5_5_07L_W4C4A2_joint_7']}</param>
                 </state_interface>
-                <state_interface name="velocity"/>
+                <state_interface name="velocity" />
             </joint>
             <joint name="lh_index_mcp_pitch">
-                <command_interface name="position"/>
+                <command_interface name="position" />
                 <state_interface name="position">
                   <param name="initial_value">${initial_positions['lh_index_mcp_pitch']}</param>
                 </state_interface>
-                <state_interface name="velocity"/>
+                <state_interface name="velocity" />
             </joint>
             <joint name="lh_middle_mcp_pitch">
-                <command_interface name="position"/>
+                <command_interface name="position" />
                 <state_interface name="position">
                   <param name="initial_value">${initial_positions['lh_middle_mcp_pitch']}</param>
                 </state_interface>
-                <state_interface name="velocity"/>
+                <state_interface name="velocity" />
             </joint>
             <joint name="lh_pinky_mcp_pitch">
-                <command_interface name="position"/>
+                <command_interface name="position" />
                 <state_interface name="position">
                   <param name="initial_value">${initial_positions['lh_pinky_mcp_pitch']}</param>
                 </state_interface>
-                <state_interface name="velocity"/>
+                <state_interface name="velocity" />
             </joint>
             <joint name="lh_ring_mcp_pitch">
-                <command_interface name="position"/>
+                <command_interface name="position" />
                 <state_interface name="position">
                   <param name="initial_value">${initial_positions['lh_ring_mcp_pitch']}</param>
                 </state_interface>
-                <state_interface name="velocity"/>
+                <state_interface name="velocity" />
             </joint>
             <joint name="lh_thumb_cmc_yaw">
-                <command_interface name="position"/>
+                <command_interface name="position" />
                 <state_interface name="position">
                   <param name="initial_value">${initial_positions['lh_thumb_cmc_yaw']}</param>
                 </state_interface>
-                <state_interface name="velocity"/>
+                <state_interface name="velocity" />
             </joint>
             <joint name="lh_thumb_cmc_pitch">
-                <command_interface name="position"/>
+                <command_interface name="position" />
                 <state_interface name="position">
                   <param name="initial_value">${initial_positions['lh_thumb_cmc_pitch']}</param>
                 </state_interface>
-                <state_interface name="velocity"/>
+                <state_interface name="velocity" />
             </joint>
-        </ros2_control>
+        <joint name="lh_thumb_ip"><param name="mimic">lh_thumb_cmc_pitch</param><param name="multiplier">2.29</param><state_interface name="position" /><state_interface name="velocity" /></joint><joint name="lh_index_dip"><param name="mimic">lh_index_mcp_pitch</param><param name="multiplier">0.89</param><state_interface name="position" /><state_interface name="velocity" /></joint><joint name="lh_middle_dip"><param name="mimic">lh_middle_mcp_pitch</param><param name="multiplier">0.89</param><state_interface name="position" /><state_interface name="velocity" /></joint><joint name="lh_ring_dip"><param name="mimic">lh_ring_mcp_pitch</param><param name="multiplier">0.89</param><state_interface name="position" /><state_interface name="velocity" /></joint><joint name="lh_pinky_dip"><param name="mimic">lh_pinky_mcp_pitch</param><param name="multiplier">0.89</param><state_interface name="position" /><state_interface name="velocity" /></joint></ros2_control>
     </xacro:macro>
 </robot>
